File: m48t59y.kicad_sch (KiCad schematic)
At the start: 3 parts, among them U4 74HC595, U5 74HC595, U7 M48T08-150PC

Commit message: Update schematics, PCB, and add fp-lib-table
Parts:
- removed U4, U5: 74HC595, Package_SO:SOIC-16_3.9x9.9mm_P1.27mm, symbol 74xx:74HC595
- U7: footprint Package_DIP:DIP-28_W15.24mm -> kicad:DIP-28_W15.24mm
Connections:
- net A8: now reaches U7.25 (A8)
- net Q1A renamed A7
- net Q1B renamed A6
- net Q1C renamed A5
- net Q1D renamed A4
- net Q1E renamed A3
- net Q1F renamed A2
- net Q1G renamed A1
- net Q1H renamed A0
- net Q2B renamed A12
- net Q2C renamed A9
- net Q2D renamed A11
- net Q2E renamed A10
