File: m48t59y_pic18f.kicad_sch (KiCad schematic)
At the start: 0 parts

Commit message: Update schematics, PCB, and add fp-lib-table
Other:
- sheet RaspberryPi4 ports: added GPIO10, GPIO11, GPIO9; removed MISO, MOSI, SCLK
- sheet m48t59y ports: added A0, A1, A10, A11, A12, A2, A3, A4, A5, A6, A7, A8, A9; removed RCLK, SER_IN, SRCCLK
- sheet txs0108e ports: added A1C, A2C, A3C, A4C, A5C, A6C, A7C, A8C, B1C, B2C, B3C, B4C, B5C, B6C, B7C, B8C; removed none
