File: mcu.kicad_sch (KiCad schematic)
At the start: 3 parts, among them J4 Raspberry_Pi_4

Commit message: Update schematics, PCB, and add fp-lib-table
Parts:
- J4: footprint Connector_PinHeader_2.54mm:PinHeader_2x20_P2.54mm_Vertical -> kicad:PinHeader_2x20_P2.54mm_Vertical
Connections:
- net MISO renamed GPIO9
- net MOSI renamed GPIO10
- net SCLK renamed GPIO11
Changed lines of the file:
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@@
 		)
 	)
-	(hierarchical_label "MISO"
+	(hierarchical_label "GPIO9"
 		(shape input)
 		(at 196.85 107.95 0)
@@
 		)
 	)
-	(hierarchical_label "SCLK"
+	(hierarchical_label "GPIO11"
 		(shape input)
 		(at 196.85 113.03 0)
@@
 		)
 	)
-	(hierarchical_label "MOSI"
+	(hierarchical_label "GPIO10"
 		(shape input)
 		(at 196.85 110.49 0)
@@
 			)
 		)
-		(property "Footprint" "Connector_PinHeader_2.54mm:PinHeader_2x20_P2.54mm_Vertical"
+		(property "Footprint" "kicad:PinHeader_2x20_P2.54mm_Vertical"
 			(at 233.934 140.208 0)
 			(hide yes)
