File: txs0108e.kicad_sch (KiCad schematic)
At the start: 2 parts, among them U1 TXS0108, U2 TXS0108

Commit message: Update schematics, PCB, and add fp-lib-table
Parts:
- added U4: TXS0108, kicad:TXS0108E_THT_20pin_big, symbol txs0108:TXS0108
- U1, U2: footprint kiC:TXS0108E_THT_20pin -> kicad:TXS0108E_THT_20pin_big
Connections:
- net +3V3: now also U4.1 (VCCA)
- net +5V: now also U4.20 (VCCB)
- net GND: now also U4.11 (GND)
- net OE: now also U4.10 (OE)
- new net A1C: U4.2 (A1)
- new net A2C: U4.3 (A2)
- new net A3C: U4.4 (A3)
- new net A4C: U4.5 (A4)
- new net A5C: U4.6 (A5)
- new net A6C: U4.7 (A6)
- new net A7C: U4.8 (A7)
- new net A8C: U4.9 (A8)
- new net B1C: U4.19 (B1)
- new net B2C: U4.18 (B2)
- new net B3C: U4.17 (B3)
- new net B4C: U4.16 (B4)
- new net B5C: U4.15 (B5)
- new net B6C: U4.14 (B6)
- new net B7C: U4.13 (B7)
- new net B8C: U4.12 (B8)
